Commit message: MapMyWorld Project V1.0

File: src/my_robot/urdf/my_robot.xacro (robot description, xacro)
@@ -194,3 +194,10 @@
   </visual>
  </link>
+ <joint name="camera_optical_joint" type="fixed">
+  <origin xyz="0 0 0" rpy="-1.5705 0 -1.5707"/>
+  <parent link="camera"/>
+  <child link="camera_link_optical"/>
+ </joint>
+ <link name="camera_link_optical">
+ </link>
 </robot>
